File: espilepsy.kicad_sch (KiCad schematic)
At the start: 27 parts, among them J1 Conn_01x06, J2 Screw_Terminal_01x02, J3 Screw_Terminal_01x02, J4 Screw_Terminal_01x02, J5 Screw_Terminal_01x02, Q1 BSS138, Q2 IRF9310, SW1 SW_Push, U1 NCP1117-3.3_SOT223, U3 ESP32-WROOM-32D

Commit message: Build v1
Parts:
- removed R2: R, Resistor_SMD:R_0603_1608Metric_Pad0.98x0.95mm_HandSolder, symbol Device:R
- removed R3: 0, Resistor_SMD:R_0603_1608Metric_Pad0.98x0.95mm_HandSolder, symbol Device:R
- removed SW1: SW_Push, Button_Switch_SMD:SW_Push_1P1T_NO_6x6mm_H9.5mm, symbol Switch:SW_Push
- added H1, H2: MountingHole, MountingHole:MountingHole_2.7mm_M2.5, symbol Mechanical:MountingHole
- added J6: Conn_01x02_Pin, Connector_PinHeader_2.54mm:PinHeader_1x02_P2.54mm_Vertical, symbol Connector:Conn_01x02_Pin
- F1: footprint Fuse:Fuseholder_Clip-5x20mm_Keystone_3512P_Inline_P23.62x7.27mm_D1.02x2.41x1.02x1.57mm_Horizontal -> Fuse:Fuseholder_Clip-5x20mm_Littelfuse_520_Inline_P20.50x5.80mm_D1.30mm_Horizontal
- J2, J3, J4, J5: footprint TerminalBlock_MetzConnect:TerminalBlock_MetzConnect_Type073_RT02602HBLU_1x02_P5.08mm_Horizontal -> Library:TerminalBlock_MetzConnect_Type073_RT02602HBLU_1x02_P5.08mm_Horizontal_mod
Connections:
- net IO22 is gone; now on net BTN_1: U3.36 (IO22)
- net BTN_1: now also J6.2 (Pin_2); no longer U3.33 (IO21)
- net GND: now also J1.6 (Pin_6), U1.1 (ADJ), J6.1 (Pin_1); no longer J1.5 (Pin_5)
- net IO0: now also J1.5 (Pin_5); no longer J1.6 (Pin_6)
- net VIN: now reaches F1.2, J5.2 (Pin_2)
- net IO23: no longer names the net of U3.37 (IO23)
- no-connect marks 18 -> 21
Other:
- moved on the sheet: F1, TP2, TP3
